File: driver_bts7960_v1/driver_bts7960_v1.kicad_pcb (KiCad board)
At the start: 2 copper layers, 50.3 x 45 mm, 32 parts, among them J1 Motor_1, J2 XT30, J3 Conn_01x08_Pin, J6 Motor_2, U1 BTS7960B, U2 BTS7960B, U3 BTS7960B, U4 BTS7960B, U5 74HC244

Commit message: cnc
Parts:
- moved C4 0.16 mm to (156.2, 59.1)
Routing:
- net OUT_EN_2: track 43.8 -> 42.5 mm
- net GND: track 200.2 -> 198.9 mm
- net OUT_C: track 5.89 -> 5.23 mm
