File: driver_bts7960_v1/driver_bts7960_v1.kicad_pcb (KiCad board)
At the start: 2 copper layers, 50.3 x 45 mm, 32 parts, among them J1 Motor_1, J2 XT30, J3 Conn_01x08_Pin, J6 Motor_2, U1 BTS7960B, U2 BTS7960B, U3 BTS7960B, U4 BTS7960B, U5 74HC244

Commit message: Version final (sin archivos 3D)
Parts:
- added G***: LOGO, AidenMaidPerez:LogoAidenMP_Neg, F.Cu at (117.8, 70.7)
Other:
- board text added: "Designed by Aiden Maid Pérez - 2026 CC BY-NC-SA 4.0"
- board text added: "TITANCORE 7960"
- board text removed: "2026"
- board text removed: "Aiden MP"

Commit message: .
Parts:
- C1, C2, C3, C4: value 470nF -> 100nF
- C5: footprint Capacitor_THT:CP_Radial_D8.0mm_P3.80mm -> Capacitor_THT:CP_Radial_D8.0mm_P5.00mm
- R1, R10, R2, R3, R4, R5, R6, R7, R8, R9: value R_US -> 10k
- R11, R12, R13, R14: value R_US -> 30k
- moved C5 0.40 mm to (157.0, 66.2)
Connections:
- net +24V renamed VS
- net +5V renamed VCC
