File: driver_bts7960_v1/driver_bts7960_v1.kicad_sch (KiCad schematic)
At the start: 28 parts, among them J1 Motor_1, J2 XT30, J3 Conn_01x08_Pin, J6 Motor_2, U1 BTS7960B, U2 BTS7960B, U3 BTS7960B, U4 BTS7960B, U5 74HC244

Commit message: version funcional y con valores de componentes
Parts:
- C1, C2, C3, C4: value 470nF -> 100nF
- R1, R10, R2, R3, R4, R5, R6, R7, R8, R9: value R_US -> 10k
- R11, R12, R13, R14: value R_US -> 30k
Changed lines of the file:
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@@
 			)
 		)
-		(property "Value" "R_US"
+		(property "Value" "10k"
 			(at 91.44 32.766 90)
 			(show_name no)
@@
 			)
 		)
-		(property "Value" "R_US"
+		(property "Value" "30k"
 			(at 91.44 37.846 90)
 			(show_name no)
@@
 			)
 		)
-		(property "Value" "R_US"
+		(property "Value" "30k"
 			(at 91.44 67.056 90)
 			(show_name no)
@@
 			)
 		)
-		(property "Value" "R_US"
+		(property "Value" "10k"
 			(at 91.44 123.952 90)
 			(show_name no)
@@
 			)
 		)
-		(property "Value" "470nF"
+		(property "Value" "100nF"
 			(at 133.858 30.988 0)
 			(show_name no)
@@
 			)
 		)
-		(property "Value" "R_US"
+		(property "Value" "10k"
 			(at 137.16 129.5399 0)
 			(show_name no)
@@
 			)
 		)
-		(property "Value" "R_US"
+		(property "Value" "10k"
 			(at 91.44 117.094 90)
 			(show_name no)
@@
 			)
 		)
-		(property "Value" "470nF"
+		(property "Value" "100nF"
 			(at 134.874 59.944 0)
 			(show_name no)
@@
 			)
 		)
-		(property "Value" "R_US"
+		(property "Value" "30k"
 			(at 91.44 100.076 90)
 			(show_name no)
@@
 			)
 		)
-		(property "Value" "470nF"
+		(property "Value" "100nF"
 			(at 133.858 93.218 0)
 			(show_name no)
@@
 			)
 		)
-		(property "Value" "470nF"
+		(property "Value" "100nF"
 			(at 134.874 122.174 0)
 			(show_name no)
@@
 			)
 		)
-		(property "Value" "R_US"
+		(property "Value" "10k"
 			(at 91.44 88.392 90)
 			(show_name no)
@@
 			)
 		)
-		(property "Value" "R_US"
+		(property "Value" "10k"
 			(at 91.44 94.996 90)
 			(show_name no)
@@
 			)
 		)
-		(property "Value" "R_US"
+		(property "Value" "10k"
 			(at 91.44 54.864 90)
 			(show_name no)
@@
 			)
 		)
-		(property "Value" "R_US"
+		(property "Value" "30k"
 			(at 91.44 129.032 90)
 			(show_name no)
@@
 			)
 		)
-		(property "Value" "R_US"
+		(property "Value" "10k"
 			(at 91.44 61.722 90)
 			(show_name no)
@@
 			)
 		)
-		(property "Value" "R_US"
+		(property "Value" "10k"
 			(at 137.16 67.3099 0)
 			(show_name no)
@@
 			)
 		)
-		(property "Value" "R_US"
+		(property "Value" "10k"
 			(at 91.44 26.162 90)
 			(show_name no)
