File: driver_bts7960_v1/driver_bts7960_v1.kicad_sch (KiCad schematic)
At the start: 28 parts, among them J1 Motor_1, J2 XT30, J3 Conn_01x08_Pin, J6 Motor_2, U1 BTS7960B, U2 BTS7960B, U3 BTS7960B, U4 BTS7960B, U5 74HC244

Commit message: Version final (sin archivos 3D)
Connections:
- net +24V renamed VS
- net +5V renamed VCC
Other:
- note added: "Designed by Aiden Maid Pérez - 2026 CC BY-NC-SA 4.0"

Commit message: .
Parts:
- C5: footprint Capacitor_THT:CP_Radial_D8.0mm_P3.80mm -> Capacitor_THT:CP_Radial_D8.0mm_P5.00mm
Changed lines of the file:
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@@
 			)
 		)
-		(property "Footprint" "Capacitor_THT:CP_Radial_D8.0mm_P3.80mm"
+		(property "Footprint" "Capacitor_THT:CP_Radial_D8.0mm_P5.00mm"
 			(at 40.3352 29.21 0)
 			(hide yes)

Commit message: .
Other:
- note added: "(c) 2026 Aiden Maid Pérez - CC BY-NC-SA 4.0"
- note removed: "Designed by Aiden Maid Pérez - 2026 CC BY-NC-SA 4.0"
- company: (none) -> Aiden Maid Pérez
- title: (none) -> TitanCore-7960 Dual Motor Driver
Changed lines of the file:
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@@
 	(generator_version "10.0")
 	(paper "A4")
-	(rectangle
-		(start 12.7 115.57)
-		(end 63.5 137.16)
-		(stroke
-			(width 0)
-			(type default)
-		)
-		(fill
-			(type none)
-		)
+	(title_block
+		(title "TitanCore-7960 Dual Motor Driver")
+		(company "Aiden Maid Pérez")
+		(comment 1 "Licensed under CC BY-NC-SA 4.0")
 	)
 	(rectangle
@@
 		)
 	)
-	(text "Designed by Aiden Maid Pérez - 2026\nCC BY-NC-SA 4.0"
+	(text "(c) 2026 Aiden Maid Pérez - CC BY-NC-SA 4.0"
 		(exclude_from_sim no)
-		(at 14.224 133.096 0)
+		(at 112.522 139.446 0)
 		(effects
 			(font
